File: Electronics/LightTouch_10x10/LightTouch_10x10.kicad_pcb (KiCad board)
At the start: 2 copper layers, 100 x 100 mm, 400 parts, among them Q1 RPM-075PTT86, Q10 RQ5E070BNTCL, Q100 RQ5E070BNTCL, Q101 RPM-075PTT86, Q102 RQ5E070BNTCL, Q103 RPM-075PTT86, Q104 RQ5E070BNTCL, Q105 RPM-075PTT86, Q106 RQ5E070BNTCL, Q107 RPM-075PTT86, Q108 RQ5E070BNTCL, Q109 RPM-075PTT86, Q11 RPM-075PTT86, Q110 RQ5E070BNTCL, Q111 RPM-075PTT86, Q112 RQ5E070BNTCL, Q113 RPM-075PTT86, Q114 RQ5E070BNTCL, Q115 RPM-075PTT86, Q116 RQ5E070BNTCL, Q117 RPM-075PTT86, Q118 RQ5E070BNTCL, Q119 RPM-075PTT86, Q12 RQ5E070BNTCL, Q120 RQ5E070BNTCL, Q121 RPM-075PTT86, Q122 RQ5E070BNTCL, Q123 RPM-075PTT86, Q124 RQ5E070BNTCL, Q125 RPM-075PTT86, Q126 RQ5E070BNTCL, Q127 RPM-075PTT86, Q128 RQ5E070BNTCL, Q129 RPM-075PTT86, Q13 RPM-075PTT86, Q130 RQ5E070BNTCL, Q131 RPM-075PTT86, Q132 RQ5E070BNTCL, Q133 RPM-075PTT86, Q134 RQ5E070BNTCL, Q135 RPM-075PTT86, Q136 RQ5E070BNTCL, Q137 RPM-075PTT86, Q138 RQ5E070BNTCL, Q139 RPM-075PTT86, Q14 RQ5E070BNTCL, Q140 RQ5E070BNTCL, Q141 RPM-075PTT86, Q142 RQ5E070BNTCL, Q143 RPM-075PTT86, Q144 RQ5E070BNTCL, Q145 RPM-075PTT86, Q146 RQ5E070BNTCL, Q147 RPM-075PTT86, Q148 RQ5E070BNTCL, Q149 RPM-075PTT86, Q15 RPM-075PTT86, Q150 RQ5E070BNTCL, Q151 RPM-075PTT86, Q152 RQ5E070BNTCL, Q153 RPM-075PTT86, Q154 RQ5E070BNTCL, Q155 RPM-075PTT86, Q156 RQ5E070BNTCL, Q157 RPM-075PTT86, Q158 RQ5E070BNTCL, Q159 RPM-075PTT86, Q16 RQ5E070BNTCL, Q160 RQ5E070BNTCL, Q161 RPM-075PTT86, Q162 RQ5E070BNTCL, Q163 RPM-075PTT86, Q164 RQ5E070BNTCL, Q165 RPM-075PTT86, Q166 RQ5E070BNTCL, Q167 RPM-075PTT86, Q168 RQ5E070BNTCL, Q169 RPM-075PTT86, Q17 RPM-075PTT86, Q170 RQ5E070BNTCL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

Commit message: Added silkscreen layer
Other:
- board text added: "RE TOUCH"
Changed lines of the file:
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@@
 		(layer "Edge.Cuts")
+	)
+	(gr_text "RE TOUCH"
+		(at 192 151 0)
+		(layer "F.SilkS")
+		(effects
+			(font
+				(size 1 1)
+				(thickness 0.1)
+			)
+			(justify left bottom)
+		)
+	)
+	(gr_text "RE TOUCH"
+		(at 110 151 0)
+		(layer "B.SilkS")
+		(effects
+			(font
+				(size 1 1)
+				(thickness 0.1)
+			)
+			(justify left bottom mirror)
+		)
 	)
 	(via
